File: regulator.sch (KiCad schematic (older format))
At the start: 5 parts, among them IC1 MAX20029ATIC_V+

Commit message: Update schematic sheets
Parts:
- IC1: symbol Simple_SDR-rescue:MAX20029ATIC_V+-MAX20029ATIC_V+ -> MAX20029ATIC_V+:MAX20029ATIC_V+
Changed lines of the file:
@@
 $EndDescr
 $Comp
-L Simple_SDR-rescue:MAX20029ATIC_V+-MAX20029ATIC_V+ IC1
+L MAX20029ATIC_V+:MAX20029ATIC_V+ IC1
 U 1 1 675F18F2
 P 4400 3650

Commit message: Update regulator.sch after changing MAX part ID
Parts:
- IC1: value MAX20029ATIC_V+ -> MAX20029ATIF_V+; symbol MAX20029ATIC_V+:MAX20029ATIC_V+ -> MAX20029ATIF_V+:MAX20029ATIC_V+
Changed lines of the file:
@@
 $Descr A4 11693 8268
 encoding utf-8
-Sheet 7 7
+Sheet 6 7
 Title ""
 Date ""
@@
 $EndDescr
 $Comp
-L MAX20029ATIC_V+:MAX20029ATIC_V+ IC1
+L MAX20029ATIF_V+:MAX20029ATIC_V+ IC1
 U 1 1 675F18F2
 P 4400 3650
@@
 AR Path="/675F00E9/675F18F2" Ref="IC1"  Part="1"
 F 0 "IC1" H 5550 4350 50  0000 L CNN
-F 1 "MAX20029ATIC_V+" H 5550 4450 50  0000 L CNN
+F 1 "MAX20029ATIF_V+" H 5550 4450 50  0000 L CNN
 F 2 "Package_DFN_QFN:TQFN-28-1EP_5x5mm_P0.5mm_EP2.7x2.7mm" H 5550 4150 50  0001 L CNN
 F 3 "https://www.mouser.jp/datasheet/2/256/Maxim_MAX20029-29B_DS_(Rev_11_2c_prelim)-1830034.pdf" H 5550 4050 50  0001 L CNN

Commit message: Create new sheet for DDR3L schematic
Parts:
- added L?: 1u5, symbol Device:L
Changed lines of the file:
@@
 $Descr A4 11693 8268
 encoding utf-8
-Sheet 6 7
+Sheet 6 8
 Title ""
 Date ""
@@
 	3450 2750 4050 2750
 Connection ~ 4050 2750
+$Comp
+L Device:L L?
+U 1 1 675F5ED4
+P 6300 3300
+F 0 "L?" V 6490 3300 50  0000 C CNN
+F 1 "1u5" V 6399 3300 50  0000 C CNN
+F 2 "" H 6300 3300 50  0001 C CNN
+F 3 "~" H 6300 3300 50  0001 C CNN
+	1    6300 3300
+	0    -1   -1   0
+$EndComp
 $EndSCHEMATC
