File: zynq_pl.sch (KiCad schematic (older format))
At the start: 1 part

Commit message: Add regulator page and rework its symbol footprint
Parts:
- U1: renamed from U?; footprint BGA225C80P15X15_1300X1300X150 -> Package_BGA:Xilinx_CLG225; symbol XC7Z007S-1CLG225C:XC7Z007S-1CLG225C -> Simple_SDR-rescue:XC7Z007S-1CLG225C-XC7Z007S-1CLG225C
Changed lines of the file:
@@
 $Descr A4 11693 8268
 encoding utf-8
-Sheet 3 6
+Sheet 3 7
 Title ""
 Date ""
@@
 $EndDescr
 $Comp
-L XC7Z007S-1CLG225C:XC7Z007S-1CLG225C U?
+L Simple_SDR-rescue:XC7Z007S-1CLG225C-XC7Z007S-1CLG225C U1
 U 5 1 67607CC2
 P 4400 3350
-F 0 "U?" H 4400 4915 50  0000 C CNN
+F 0 "U1" H 4400 4915 50  0000 C CNN
 F 1 "XC7Z007S-1CLG225C" H 4400 4824 50  0000 C CNN
-F 2 "BGA225C80P15X15_1300X1300X150" H 4400 3350 50  0001 L BNN
+F 2 "Package_BGA:Xilinx_CLG225" H 4400 3350 50  0001 L BNN
 F 3 "" H 4400 3350 50  0001 L BNN
 F 4 "Xilinx Inc." H 4400 3350 50  0001 L BNN "MF"

Commit message: Update schematic sheets
Parts:
- U1: symbol Simple_SDR-rescue:XC7Z007S-1CLG225C-XC7Z007S-1CLG225C -> XC7Z007S-1CLG225C:XC7Z007S-1CLG225C
Changed lines of the file:
@@
 $EndDescr
 $Comp
-L Simple_SDR-rescue:XC7Z007S-1CLG225C-XC7Z007S-1CLG225C U1
-U 5 1 67607CC2
+L XC7Z007S-1CLG225C:XC7Z007S-1CLG225C U1
+U 1 1 67607CC2
 P 4400 3350
 F 0 "U1" H 4400 4915 50  0000 C CNN
@@
 F 15 "Bad" H 4400 3350 50  0001 L BNN "AVAILABILITY"
 F 16 "Xilinx" H 4400 3350 50  0001 L BNN "MANUFACTURER"
-	5    4400 3350
+	1    4400 3350
 	1    0    0    -1
 $EndComp
