File: zynq_power.sch (KiCad schematic (older format))
At the start: 1 part

Commit message: Add regulator page and rework its symbol footprint
Parts:
- U1: renamed from U?; footprint BGA225C80P15X15_1300X1300X150 -> Package_BGA:Xilinx_CLG225; symbol XC7Z007S-1CLG225C:XC7Z007S-1CLG225C -> Simple_SDR-rescue:XC7Z007S-1CLG225C-XC7Z007S-1CLG225C
Changed lines of the file:
@@
 $Descr A4 11693 8268
 encoding utf-8
-Sheet 4 6
+Sheet 4 7
 Title ""
 Date ""
@@
 $EndDescr
 $Comp
-L XC7Z007S-1CLG225C:XC7Z007S-1CLG225C U?
+L Simple_SDR-rescue:XC7Z007S-1CLG225C-XC7Z007S-1CLG225C U1
 U 1 1 675E564F
 P 3250 2750
-F 0 "U?" H 3300 4115 50  0000 C CNN
+F 0 "U1" H 3300 4115 50  0000 C CNN
 F 1 "XC7Z007S-1CLG225C" H 3300 4024 50  0000 C CNN
-F 2 "BGA225C80P15X15_1300X1300X150" H 3250 2750 50  0001 L BNN
+F 2 "Package_BGA:Xilinx_CLG225" H 3250 2750 50  0001 L BNN
 F 3 "" H 3250 2750 50  0001 L BNN
 F 4 "Xilinx Inc." H 3250 2750 50  0001 L BNN "MF"

Commit message: Update schematic sheets
Parts:
- U1: symbol Simple_SDR-rescue:XC7Z007S-1CLG225C-XC7Z007S-1CLG225C -> XC7Z007S-1CLG225C:XC7Z007S-1CLG225C
Changed lines of the file:
@@
 $EndDescr
 $Comp
-L Simple_SDR-rescue:XC7Z007S-1CLG225C-XC7Z007S-1CLG225C U1
+L XC7Z007S-1CLG225C:XC7Z007S-1CLG225C U1
 U 1 1 675E564F
 P 3250 2750
