File: zynq_ps.sch (KiCad schematic (older format))
At the start: 1 part

Commit message: Add regulator page and rework its symbol footprint
Parts:
- U1: renamed from U?; footprint BGA225C80P15X15_1300X1300X150 -> Package_BGA:Xilinx_CLG225; symbol XC7Z007S-1CLG225C:XC7Z007S-1CLG225C -> Simple_SDR-rescue:XC7Z007S-1CLG225C-XC7Z007S-1CLG225C
Changed lines of the file:
@@
 $Descr A4 11693 8268
 encoding utf-8
-Sheet 2 6
+Sheet 2 7
 Title ""
 Date ""
@@
 $EndDescr
 $Comp
-L XC7Z007S-1CLG225C:XC7Z007S-1CLG225C U?
+L Simple_SDR-rescue:XC7Z007S-1CLG225C-XC7Z007S-1CLG225C U1
 U 4 1 675DABA9
 P 2450 2750
-F 0 "U?" H 2400 4315 50  0000 C CNN
+F 0 "U1" H 2400 4315 50  0000 C CNN
 F 1 "XC7Z007S-1CLG225C" H 2400 4224 50  0000 C CNN
-F 2 "BGA225C80P15X15_1300X1300X150" H 2450 2750 50  0001 L BNN
+F 2 "Package_BGA:Xilinx_CLG225" H 2450 2750 50  0001 L BNN
 F 3 "" H 2450 2750 50  0001 L BNN
 F 4 "Xilinx Inc." H 2450 2750 50  0001 L BNN "MF"

Commit message: Update schematic sheets
Parts:
- U1: symbol Simple_SDR-rescue:XC7Z007S-1CLG225C-XC7Z007S-1CLG225C -> XC7Z007S-1CLG225C:XC7Z007S-1CLG225C
Changed lines of the file:
@@
 $EndDescr
 $Comp
-L Simple_SDR-rescue:XC7Z007S-1CLG225C-XC7Z007S-1CLG225C U1
-U 4 1 675DABA9
+L XC7Z007S-1CLG225C:XC7Z007S-1CLG225C U1
+U 1 1 675DABA9
 P 2450 2750
 F 0 "U1" H 2400 4315 50  0000 C CNN
@@
 F 15 "Bad" H 2450 2750 50  0001 L BNN "AVAILABILITY"
 F 16 "Xilinx" H 2450 2750 50  0001 L BNN "MANUFACTURER"
-	4    2450 2750
+	1    2450 2750
 	1    0    0    -1
 $EndComp
