File: Simple_SDR.kicad_pcb (KiCad board)
At the start: 2 copper layers, 2 parts, among them IC1 MAX20029ATIC_V+, U1 XC7Z007S-1CLG225C

Commit message: Update project files
Other:
- net class Default removed
